File: usbAudio.kicad_pcb (KiCad board)
At the start: 2 copper layers, 38 parts, among them J2 USB_C_Receptacle_USB2.0_14P, J3 AudioJack3, SW1 PLAY/PAUSE, SW2 NEXT TR., SW3 MUTE, SW4 VOL+, SW5 VOL-, SW6 PREV. TR., SW7 STOP, SW8 SW_SPDT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

Commit message: Layout time!!!
Parts:
- removed SW3: MUTE, Button_Switch_THT:SW_PUSH_6mm_H4.3mm
- removed SW6: PREV. TR., Button_Switch_THT:SW_PUSH_6mm_H4.3mm
- removed SW7: STOP, Button_Switch_THT:SW_PUSH_6mm_H4.3mm
- J3: footprint Connector_Audio:Jack_3.5mm_KoreanHropartsElec_PJ-320D-4A_Horizontal -> customJack:Jack_3.5mm_KoreanHropartsElec_PJ-320D-4A_Horizontal_copy
- SW8: footprint Button_Switch_THT:SW_PUSH_6mm_H4.3mm -> JS102011SAQN:SW_JS102011SAQN
- moved SW8 107.4 mm to (167.1, 90.3), turned to 90 degrees
- moved R10 93.6 mm to (147.3, 124.2), turned to 90 degrees
- moved J2 87.1 mm to (140.7, 127.4)
- moved C22 84.4 mm to (141.0, 117.2)
- moved C4 83.7 mm to (144.8, 95.0), turned to -90 degrees
- moved R1 83.6 mm to (155.3, 81.0), turned to 180 degrees
- moved R2 82.2 mm to (155.3, 79.0), turned to 180 degrees
- moved C21 81.6 mm to (140.7, 110.1), turned to 180 degrees
- moved R12 80.9 mm to (134.1, 124.2), turned to 90 degrees
- moved C8 80.1 mm to (148.6, 82.3), turned to -90 degrees
- moved C6 78.8 mm to (147.3, 59.1), turned to 90 degrees
- moved R4 76.2 mm to (152.4, 68.1), turned to 180 degrees
- moved C5 75.5 mm to (136.7, 95.0), turned to 90 degrees
- moved C7 73.6 mm to (138.4, 59.1), turned to 90 degrees
- moved C9 72.3 mm to (143.0, 75.2)
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Routing:
- net GND: track 0.00 -> 112.4 mm
- net Net-(J2-D+-PadA6): track 0.00 -> 56.6 mm, vias 0 -> 2
- net Net-(J2-D--PadA7): track 0.00 -> 53.4 mm, vias 0 -> 3
- net Vbus: track 0.00 -> 28.8 mm, vias 0 -> 2
- net +3.3V: track 0.00 -> 24.4 mm
- net VoutL: track 0.00 -> 21.8 mm
- net VoutR: track 0.00 -> 20.2 mm
- net /RightOut: track 0.00 -> 18.2 mm
- net Net-(U1-XTI): track 0.00 -> 14.2 mm
- net /LeftOut: track 0.00 -> 12.2 mm
- net Net-(U1-XTO): track 0.00 -> 10.5 mm
- net Net-(U1-D+): track 0.00 -> 9.89 mm
- net Net-(U1-D-): track 0.00 -> 9.82 mm
- net Net-(J2-CC1): track 0.00 -> 6.82 mm
- net Net-(J2-CC2): track 0.00 -> 6.50 mm
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- added copper zone on F.Cu, net Vbus

Commit message: Make more dense!!!!
Parts:
- removed SW2: NEXT TR., Button_Switch_THT:SW_PUSH_6mm_H4.3mm
- SW8: moved to B.Cu
- moved SW1 76.7 mm to (119.5, 83.9)
- moved SW4 73.4 mm to (119.7, 93.0)
- moved SW5 73.4 mm to (119.7, 101.6)
- moved SW8 55.9 mm to (111.5, 95.9)
- moved C22 16.6 mm to (131.9, 103.3), turned to -90 degrees
- moved C5 16.1 mm to (149.6, 104.5), turned to 180 degrees
- moved C6 15.8 mm to (147.6, 74.8)
- moved R6 15.8 mm to (148.6, 80.0)
- moved R8 15.8 mm to (148.5, 67.6)
- moved C3 15.8 mm to (148.6, 83.8)
- moved R4 15.8 mm to (152.7, 83.8)
- moved R11 14.7 mm to (142.5, 104.1), turned to 0 degrees
- moved J2 13.1 mm to (141.1, 114.4)
- moved R10 13.1 mm to (147.7, 111.1)
- moved R12 13.1 mm to (134.5, 111.1)
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Connections:
- U1 pad 3: Vbus -> +3.3V
- U1 pad 5: Net-(U1-FUNC0) -> unconnected-(U1-FUNC0-Pad5)
Routing:
- net Suspend: track 0.00 -> 55.8 mm, vias 0 -> 2
- net +3.3V: track 24.4 -> 76.7 mm, vias 0 -> 4
- net Net-(J2-D+-PadA6): track 56.6 -> 15.5 mm
- net Net-(J2-D--PadA7): track 53.4 -> 15.8 mm
- net GND: track 112.4 -> 149.2 mm
- net Net-(U1-HID2/MD): track 0.00 -> 24.5 mm
- net Net-(U1-FUNC3): track 0.00 -> 19.2 mm
- net Net-(U1-HID1/MC): track 0.00 -> 19.0 mm
- net Net-(U1-DT): track 0.00 -> 8.51 mm, vias 0 -> 2
- net /LeftOut: track 12.2 -> 18.6 mm
- net Net-(U1-XTI): track 14.2 -> 17.8 mm
- net Net-(U1-D-): track 9.82 -> 6.92 mm
- net VoutL: track 21.8 -> 19.7 mm
- net Net-(U1-XTO): track 10.5 -> 12.2 mm
- net Net-(U1-D+): track 9.89 -> 8.95 mm
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
Commit message: Made ready for production!
Parts:
- added G***: LOGO, LOGO, B.Cu at (141.4, 71.3)
- added G***: LOGO, LOGO, B.Cu at (126.0, 74.9)
- added G***: LOGO, LOGO, B.Cu at (141.0, 97.3)
- added REF**: PCBA tooling hole, JLCtooling:PCBA tooling hole, F.Cu at (119.4, 114.8)
- added REF**: PCBA tooling hole, JLCtooling:PCBA tooling hole, F.Cu at (152.4, 62.5)
- added REF**: PCBA tooling hole, JLCtooling:PCBA tooling hole, F.Cu at (152.7, 114.8)
- SW8: footprint JS102011SAQN:SW_JS102011SAQN -> JS102011SAQN:SW_JS102011SAQN_Xoverhang
- moved SW8 44.5 mm to (155.7, 90.7), turned to -90 degrees
- moved J3 23.2 mm to (124.6, 65.8), turned to 0 degrees
- moved R9 9.36 mm to (133.5, 69.1)
- moved C7 9.21 mm to (133.0, 75.7), turned to 180 degrees
- moved R7 4.77 mm to (141.5, 76.7)
- moved C2 4.77 mm to (141.2, 80.5)
- moved R3 4.25 mm to (137.2, 79.2)
- moved C3 2.33 mm to (148.6, 86.2)
- moved R4 2.33 mm to (152.7, 86.2)
- moved R8 2.33 mm to (148.5, 69.9)
- moved C6 2.33 mm to (147.6, 77.2)
- moved R6 2.33 mm to (148.6, 82.3)
Routing:
- net GND: track 149.2 -> 189.7 mm, vias 0 -> 2
- net unconnected-(J2-SHIELD-PadS1): track 0.00 -> 25.8 mm
- net Net-(J2-D+-PadA6): track 15.5 -> 29.7 mm
- net Suspend: track 55.8 -> 69.0 mm
- net Net-(J2-D--PadA7): track 15.8 -> 28.4 mm
- net /LeftOut: track 18.6 -> 26.9 mm
- net +3.3V: track 76.7 -> 82.3 mm
- net /RightOut: track 18.2 -> 21.7 mm
- net VoutR: track 20.2 -> 21.7 mm
- added copper zone on B.Cu, net +3.3V
- added copper zone on F.Cu, net +3.3V
- added copper zone on F.Cu, net GND
Other:
- board outline added: 37.4 x 56.1 mm
- board text added: "+"
- board text added: "-"
- board text added: "JLCJLCJLCJLC"
