File: usbAudio.kicad_sch (KiCad schematic)
At the start: 34 parts, among them J2 USB_C_Receptacle_USB2.0_14P, J3 AudioJack3, SW1 PLAY/PAUSE, SW4 VOL+, SW5 VOL-, SW8 SW_SPDT, U1 PCM2706CPJTR, U4 MIC5504-3.3YM5-TR, Y2 Crystal_GND24

Commit message: Made ready for production!
Parts:
- C10, C21, C22, C9: LCSC Part # (none) -> C1592
- C11, C23: LCSC Part # (none) -> C250876
- C2, C3: LCSC Part # (none) -> C107147
- C4, C5: LCSC Part # (none) -> C105621
- C6, C7: LCSC Part # (none) -> C109392
- C8: LCSC Part # (none) -> C14663
- J2: LCSC Part # (none) -> C2894897
- J3: LCSC Part # (none) -> C95562
- R1, R2: LCSC Part # (none) -> C23345
- R10, R12: LCSC Part # (none) -> C23186
- R11: LCSC Part # (none) -> C22843
- R3, R4: LCSC Part # (none) -> C25185
- R5: LCSC Part # (none) -> C22935
- R6, R7, R8, R9: LCSC Part # (none) -> C22978
- SW1, SW4, SW5: LCSC Part # (none) -> C97440
- SW8: footprint JS102011SAQN:SW_JS102011SAQN -> JS102011SAQN:SW_JS102011SAQN_Xoverhang; now not fitted; now left out of the parts list
- U1: LCSC Part # (none) -> C2651268
- U4: LCSC Part # (none) -> C88419
- Y2: LCSC Part # (none) -> C9002
